File: Hardware/SystemDesign/Op52HardwareSystemDesign/Op52HardwareSystemDesign.kicad_sch (KiCad schematic)
At the start: 9 parts, among them U1 TFT_Connector_4-000103-001, U2 PICBreakoutRevB, U3 PICBreakoutRevB, U4 PICBreakoutRevB, U5 PICBreakoutRevB, U6 PICBreakoutRevB, U7 24_Input_UCRevC, U8 TFTProcessorRevE, U9 24_Input_UCRevC

Commit message: Shoe mechanicals, Arduino updates
Connections:
- net at U7. (J8_6Pin): now also U9. (J8_6Pin)
- net at U9. (J8_6Pin): no longer U7. (J8_6Pin)
Other:
- note added: "1-15,17-24"
- note added: "25-32,Pistons1-13,blank,Ped16"
- note added: "Pedal Tx on pin 1, 19200 baud (debug leftover, works so leave it)"
- note added: "RB0 Tx RB4 Rx"
- note added: "RB4 TX"
Changed lines of the file:
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@@
+		)
+	)
+	(text "RB0 Tx\nRB4 Rx"
+		(exclude_from_sim no)
+		(at 204.47 67.31 0)
+		(effects
+			(font
+				(size 1.27 1.27)
+			)
 		)
 	)
@@
 		)
 	)
+	(text "RB4 TX"
+		(exclude_from_sim no)
+		(at 204.216 96.774 0)
+		(effects
+			(font
+				(size 1.27 1.27)
+			)
+		)
+	)
+	(text "Pedal Tx on pin 1, 19200 baud (debug leftover, works so leave it)"
+		(exclude_from_sim no)
+		(at 102.362 19.304 0)
+		(effects
+			(font
+				(size 1.27 1.27)
+			)
+		)
+	)
 	(text "MIDIExtenderRevB\nRJ:\nPin1-+V\nPin2-GND\nPin5-MIDITX+\nPin6-MIDITXDATA\n"
 		(exclude_from_sim no)
@@
 		)
 	)
+	(text "1-15,17-24"
+		(exclude_from_sim no)
+		(at 204.724 104.14 0)
+		(effects
+			(font
+				(size 1.27 1.27)
+			)
+		)
+	)
 	(text "156Trunk(6)"
 		(exclude_from_sim no)
@@
 	(text "SAMs use common wire for switch and magnets\nSo we will use Negative Common\nDrivers are SamDriver32 RevB 20190826"
 		(exclude_from_sim no)
-		(at 57.658 18.034 0)
+		(at 146.304 185.674 0)
 		(effects
 			(font
@@
 		(exclude_from_sim no)
 		(at 56.642 161.798 0)
+		(effects
+			(font
+				(size 1.27 1.27)
+			)
+		)
+	)
+	(text "25-32,Pistons1-13,blank,Ped16"
+		(exclude_from_sim no)
+		(at 214.376 82.804 0)
 		(effects
 			(font
@@
 	(wire
 		(pts
-			(xy 34.29 76.2) (xy 22.86 76.2)
-		)
-		(stroke
-			(width 0)
-			(type default)
-		)
-	)
-	(wire
-		(pts
 			(xy 185.42 82.55) (xy 176.53 82.55)
 		)
@@
 		)
 		(stroke
+			(width 0)
+			(type default)
+		)
+	)
+	(wire
+		(pts
+			(xy 22.86 76.2) (xy 34.29 76.2)
+		)
+		(stroke
